Commit message: Update code

File: my_robot/urdf/my_robot.xacro (robot description, xacro)
@@ -145,4 +145,12 @@
     <axis xyz="0 1 0" rpy="0 0 0"/>
   </joint>
+  <!-- RGBD Camera -->
+  <joint name="camera_optical_joint" type="fixed">
+      <origin xyz="0 0 0" rpy="-1.5707 0 -1.5707"/>
+      <parent link="camera"/>
+      <child link="camera_link_optical"/>
+  </joint>
+  <link name="camera_link_optical">
+  </link>
   <link name="hokuyo">
     <origin xyz="0 0 0" rpy="0 0 0"/>
